File: EnvelopeVCA/EnvelopeVCA.sch (KiCad schematic (older format))
At the start: 25 parts, among them U1 TL072

Commit message: Fixed annotations, added image
Parts:
- gave numbers to parts that had none: 10
Changed lines of the file:
@@
 	7950 4050 7950 4250
 $Comp
-L Connector:TestPoint TP?
+L Connector:TestPoint TP1
 U 1 1 60B7BD11
 P 2100 3700
-F 0 "TP?" V 2275 3925 50  0000 C CNN
+F 0 "TP1" V 2275 3925 50  0000 C CNN
 F 1 "GATE/TRIGGER IN" V 2175 3925 50  0000 C CNN
 F 2 "" H 2300 3700 50  0001 C CNN
@@
 	2100 3700 2200 3700
 $Comp
-L Device:R R?
+L Device:R R9
 U 1 1 60BA1DE9
 P 2650 4200
-F 0 "R?" V 2575 4200 50  0000 C CNN
+F 0 "R9" V 2575 4200 50  0000 C CNN
 F 1 "10k" V 2650 4200 50  0000 C CNN
 F 2 "" V 2580 4200 50  0001 C CNN
@@
 	2650 3700 2800 3700
 $Comp
-L power:GND #PWR?
+L power:GND #PWR08
 U 1 1 60BB03CC
 P 2650 4475
-F 0 "#PWR?" H 2650 4225 50  0001 C CNN
+F 0 "#PWR08" H 2650 4225 50  0001 C CNN
 F 1 "GND" H 2655 4302 50  0000 C CNN
 F 2 "" H 2650 4475 50  0001 C CNN
@@
 	2650 4350 2650 4475
 $Comp
-L Device:R R?
+L Device:R R8
 U 1 1 60BB60DB
 P 2350 3275
-F 0 "R?" V 2275 3275 50  0000 C CNN
+F 0 "R8" V 2275 3275 50  0000 C CNN
 F 1 "100k" V 2350 3275 50  0000 C CNN
 F 2 "" V 2280 3275 50  0001 C CNN
@@
 	2650 3275 2650 3700
 $Comp
-L Switch:SW_Push SW?
+L Switch:SW_Push SW1
 U 1 1 60BC4F7A
 P 1900 3275
-F 0 "SW?" H 1900 3550 50  0000 C CNN
+F 0 "SW1" H 1900 3550 50  0000 C CNN
 F 1 "MANUAL GATE BUTTON" H 1900 3450 50  0000 C CNN
 F 2 "" H 1900 3475 50  0001 C CNN
@@
 	2100 3275 2200 3275
 $Comp
-L power:+9V #PWR?
+L power:+9V #PWR07
 U 1 1 60BCA542
 P 1375 2925
-F 0 "#PWR?" H 1375 2775 50  0001 C CNN
+F 0 "#PWR07" H 1375 2775 50  0001 C CNN
 F 1 "+9V" H 1390 3098 50  0000 C CNN
 F 2 "" H 1375 2925 50  0001 C CNN
@@
 Connection ~ 7025 3375
 $Comp
-L Device:R R?
+L Device:R R10
 U 1 1 60C3052E
 P 7275 3700
-F 0 "R?" H 7175 3725 50  0000 C CNN
+F 0 "R10" H 7175 3725 50  0000 C CNN
 F 1 "1k" V 7275 3700 50  0000 C CNN
 F 2 "" V 7205 3700 50  0001 C CNN
@@
 	7425 3375 7550 3375
 $Comp
-L Connector:TestPoint TP?
+L Connector:TestPoint TP2
 U 1 1 60BE0AE7
 P 7550 3375
-F 0 "TP?" V 7725 3600 50  0000 C CNN
+F 0 "TP2" V 7725 3600 50  0000 C CNN
 F 1 "ENVELOPE OUT" V 7625 3600 50  0000 C CNN
 F 2 "" H 7750 3375 50  0001 C CNN
@@
 $EndComp
 $Comp
-L Transistor_FET:MMBFJ113 Q?
+L Transistor_FET:MMBFJ113 Q1
 U 1 1 60C4BD6B
 P 8950 4075
-F 0 "Q?" H 9140 4029 50  0000 L CNN
+F 0 "Q1" H 9140 4029 50  0000 L CNN
 F 1 "MMBFJ113" H 9140 4120 50  0000 L CNN
 F 2 "Package_TO_SOT_SMD:SOT-23" H 9150 4000 50  0001 L CIN
@@
 $EndComp
 $Comp
-L Connector:TestPoint TP?
+L Connector:TestPoint TP3
 U 1 1 60C5DCC9
 P 8625 4075
-F 0 "TP?" V 8800 4300 50  0000 C CNN
+F 0 "TP3" V 8800 4300 50  0000 C CNN
 F 1 "AUDIO IN" V 8700 4300 50  0000 C CNN
 F 2 "" H 8825 4075 50  0001 C CNN
@@
 	8625 4075 8750 4075
 $Comp
-L power:GND #PWR?
+L power:GND #PWR010
 U 1 1 60C63CD5
 P 9050 4400
-F 0 "#PWR?" H 9050 4150 50  0001 C CNN
+F 0 "#PWR010" H 9050 4150 50  0001 C CNN
 F 1 "GND" H 9055 4227 50  0000 C CNN
 F 2 "" H 9050 4400 50  0001 C CNN
@@
 	9050 4275 9050 4400
 $Comp
-L Device:C C?
+L Device:C C2
 U 1 1 60C66107
 P 9400 3700
-F 0 "C?" V 9148 3700 50  0000 C CNN
+F 0 "C2" V 9148 3700 50  0000 C CNN
 F 1 "100nF" V 9239 3700 50  0000 C CNN
 F 2 "" H 9438 3550 50  0001 C CNN
@@
 	9050 3700 9050 3875
 $Comp
-L Connector:TestPoint TP?
+L Connector:TestPoint TP4
 U 1 1 60C68B1D
 P 9650 3700
-F 0 "TP?" V 9825 3925 50  0000 C CNN
+F 0 "TP4" V 9825 3925 50  0000 C CNN
 F 1 "AUDIO OUT" V 9725 3925 50  0000 C CNN
 F 2 "" H 9850 3700 50  0001 C CNN
@@
 $EndComp
 $Comp
-L power:+9V #PWR?
+L power:+9V #PWR09
 U 1 1 60D34F7B
 P 3800 3400
-F 0 "#PWR?" H 3800 3250 50  0001 C CNN
+F 0 "#PWR09" H 3800 3250 50  0001 C CNN
 F 1 "+9V" H 3815 3573 50  0000 C CNN
 F 2 "" H 3800 3400 50  0001 C CNN
